Commit message: working!

File: implementation/end_effector/pizza_cutter_description/urdf/end_effector.urdf (robot description, URDF)
Before this commit: robot bottle_gripper, 3 links, 2 joints
Joints:
- joint left_gripper_joint: type continuous -> fixed
- joint right_gripper_joint: type continuous -> fixed

Commit message: collision up, needs tuning

File: implementation/end_effector/pizza_cutter_description/urdf/end_effector.urdf (robot description, URDF)
Before this commit: robot bottle_gripper, 3 links, 2 joints
Links:
- link left_gripper: geometry collision box size=0.15 0.02 0.15; visual mesh filename=package://end_effector_description/meshes/Claw.STL scale=0.001 0.001 0.001
- link right_gripper: geometry collision box size=0.15 0.02 0.15; visual mesh filename=package://end_effector_description/meshes/Claw.STL scale=0.001 0.001 0.001

Commit message: maybe working?

File: implementation/end_effector/pizza_cutter_description/urdf/end_effector.urdf (robot description, URDF)
Before this commit: robot bottle_gripper, 3 links, 2 joints
Links:
- link left_gripper: geometry collision box size=0.15 0.01 0.15; visual mesh filename=package://end_effector_description/meshes/Claw.STL scale=0.001 0.001 0.001
- link right_gripper: geometry collision box size=0.15 0.01 0.15; visual mesh filename=package://end_effector_description/meshes/Claw.STL scale=0.001 0.001 0.001
