Commit message: coollision working

File: implementation/ur_with_end_effector_description/urdf/ur_with_end_effector.xacro (robot description, xacro)
@@ -12,4 +12,5 @@
     <parent link="tool0"/>
     <child link="mount"/>
+    <origin xyz="-0.02 0 0.04" rpy="${0} ${-pi/2} ${pi}"/>
   </joint>
 </robot>

Commit message: bleh

File: implementation/ur_with_end_effector_description/urdf/ur_with_end_effector.xacro (robot description, xacro)
@@ -12,5 +12,5 @@
     <parent link="tool0"/>
     <child link="mount"/>
-    <origin xyz="-0.02 0 0.04" rpy="${0} ${-pi/2} ${pi}"/>
+    <origin xyz="0.02 0 0.04" rpy="${pi} ${-pi/2} ${pi}"/>
   </joint>
 </robot>
